File: Audio_Cape_B1.brd (EAGLE design)
At the start: 69.2 x 54.6 mm, 42 parts, among them U1 TLV320AIC3104, U2 V_REG_LDOSMD

Commit message: Finished Silkscreen
Parts:
- moved U$4 35.5 mm to (21.3, 8.57)
- moved U$6 13.0 mm to (21.3, 45.7)
- moved U$1 12.7 mm to (25.1, 46.4)
Other:
- board text added: "In"
- board text added: "Out"
